Commit message: observe legs waist state

File: g1_hardware/config/g1_no_hand_real.ros2_control.xacro (robot description, xacro)
@@ -17,4 +17,67 @@
                 <param name="weight_rate">${weight_rate}</param>
             </hardware>
+            <!-- Left leg joints (state-only — controlled by onboard locomotion controller) -->
+            <joint name="left_hip_pitch_joint">
+                <state_interface name="position"/>
+                <state_interface name="velocity"/>
+            </joint>
+            <joint name="left_hip_roll_joint">
+                <state_interface name="position"/>
+                <state_interface name="velocity"/>
+            </joint>
+            <joint name="left_hip_yaw_joint">
+                <state_interface name="position"/>
+                <state_interface name="velocity"/>
+            </joint>
+            <joint name="left_knee_joint">
+                <state_interface name="position"/>
+                <state_interface name="velocity"/>
+            </joint>
+            <joint name="left_ankle_pitch_joint">
+                <state_interface name="position"/>
+                <state_interface name="velocity"/>
+            </joint>
+            <joint name="left_ankle_roll_joint">
+                <state_interface name="position"/>
+                <state_interface name="velocity"/>
+            </joint>
+            <!-- Right leg joints (state-only) -->
+            <joint name="right_hip_pitch_joint">
+                <state_interface name="position"/>
+                <state_interface name="velocity"/>
+            </joint>
+            <joint name="right_hip_roll_joint">
+                <state_interface name="position"/>
+                <state_interface name="velocity"/>
+            </joint>
+            <joint name="right_hip_yaw_joint">
+                <state_interface name="position"/>
+                <state_interface name="velocity"/>
+            </joint>
+            <joint name="right_knee_joint">
+                <state_interface name="position"/>
+                <state_interface name="velocity"/>
+            </joint>
+            <joint name="right_ankle_pitch_joint">
+                <state_interface name="position"/>
+                <state_interface name="velocity"/>
+            </joint>
+            <joint name="right_ankle_roll_joint">
+                <state_interface name="position"/>
+                <state_interface name="velocity"/>
+            </joint>
+            <!-- Waist joints (state-only) -->
+            <joint name="waist_yaw_joint">
+                <state_interface name="position"/>
+                <state_interface name="velocity"/>
+            </joint>
+            <joint name="waist_roll_joint">
+                <state_interface name="position"/>
+                <state_interface name="velocity"/>
+            </joint>
+            <joint name="waist_pitch_joint">
+                <state_interface name="position"/>
+                <state_interface name="velocity"/>
+            </joint>
             <!-- Left arm joints -->
             <joint name="left_shoulder_pitch_joint">

Commit message: support waist kp kd gains

File: g1_hardware/config/g1_no_hand_real.ros2_control.xacro (robot description, xacro)
@@ -8,5 +8,5 @@
       weight_rate:      how fast (weight units/s) to ramp the arm SDK control weight.
     -->
-    <xacro:macro name="g1_ros2_control" params="name network_interface kp:=60.0 kd:=1.5 weight_rate:=0.2">
+    <xacro:macro name="g1_ros2_control" params="name network_interface kp:=60.0 kd:=1.5 waist_kp:=100.0 waist_kd:=2.0 weight_rate:=0.2">
         <ros2_control name="${name}" type="system">
             <hardware>
@@ -15,4 +15,6 @@
                 <param name="kp">${kp}</param>
                 <param name="kd">${kd}</param>
+                <param name="waist_kp">${waist_kp}</param>
+                <param name="waist_kd">${waist_kd}</param>
                 <param name="weight_rate">${weight_rate}</param>
             </hardware>

File: g1_hardware/config/g1_no_hand_real.urdf.xacro (robot description, xacro)
@@ -8,4 +8,6 @@
     <xacro:arg name="kp"          default="60.0"/>
     <xacro:arg name="kd"          default="1.5"/>
+    <xacro:arg name="waist_kp"    default="100.0"/>
+    <xacro:arg name="waist_kd"    default="2.0"/>
     <xacro:arg name="weight_rate" default="0.2"/>
     <xacro:include filename="$(find g1_description)/g1_29dof.urdf"/>
@@ -16,4 +18,6 @@
         kp="$(arg kp)"
         kd="$(arg kd)"
+        waist_kp="$(arg waist_kp)"
+        waist_kd="$(arg waist_kd)"
         weight_rate="$(arg weight_rate)"/>
 </robot>

Commit message: fix waist_kp parameter and remove weight decreasing rate parameter

File: g1_hardware/config/g1_no_hand_real.ros2_control.xacro (robot description, xacro)
@@ -8,5 +8,5 @@
       weight_rate:      how fast (weight units/s) to ramp the arm SDK control weight.
     -->
-    <xacro:macro name="g1_ros2_control" params="name network_interface kp:=60.0 kd:=1.5 waist_kp:=100.0 waist_kd:=2.0 weight_rate:=0.2">
+    <xacro:macro name="g1_ros2_control" params="name network_interface kp:=60.0 kd:=1.5 waist_kp:=200.0 waist_kd:=2.0">
         <ros2_control name="${name}" type="system">
             <hardware>
@@ -17,5 +17,4 @@
                 <param name="waist_kp">${waist_kp}</param>
                 <param name="waist_kd">${waist_kd}</param>
-                <param name="weight_rate">${weight_rate}</param>
             </hardware>
             <!-- Left leg joints (state-only — controlled by onboard locomotion controller) -->

File: g1_hardware/config/g1_no_hand_real.urdf.xacro (robot description, xacro)
@@ -8,7 +8,6 @@
     <xacro:arg name="kp"          default="60.0"/>
     <xacro:arg name="kd"          default="1.5"/>
-    <xacro:arg name="waist_kp"    default="100.0"/>
+    <xacro:arg name="waist_kp"    default="200.0"/>
     <xacro:arg name="waist_kd"    default="2.0"/>
-    <xacro:arg name="weight_rate" default="0.2"/>
     <xacro:include filename="$(find g1_description)/g1_29dof.urdf"/>
     <xacro:include filename="g1_no_hand_real.ros2_control.xacro"/>
@@ -19,5 +18,4 @@
         kd="$(arg kd)"
         waist_kp="$(arg waist_kp)"
-        waist_kd="$(arg waist_kd)"
-        weight_rate="$(arg weight_rate)"/>
+        waist_kd="$(arg waist_kd)"/>
 </robot>
