Commit message: Automatically close hands when their hardware interface is ordered to be deactivated

File: g1_hardware/config/g1_inspire_dfq_real.urdf.xacro (robot description, xacro)
@@ -14,4 +14,5 @@
   <xacro:arg name="inspire_state_topic" default="rt/inspire/state"/>
   <xacro:arg name="inspire_state_timeout_sec" default="3.0"/>
+  <xacro:arg name="close_hand_on_deactivate" default="true"/>
   <xacro:include filename="$(find g1_description)/g1_29dof_rev_1_0_with_inspire_hand_DFQ.urdf"/>
   <xacro:include filename="g1_no_hand_real.ros2_control.xacro"/>
@@ -19,4 +20,4 @@
   <xacro:include filename="inspire_rh56dfx_real.ros2_control.xacro"/>
   <xacro:g1_ros2_control name="G1RealSystem" network_interface="$(arg network_interface)" kp="$(arg kp)" kd="$(arg kd)" waist_kp="$(arg waist_kp)" waist_kd="$(arg waist_kd)"/>
-  <xacro:inspire_rh56dfx_ros2_control name="InspireRH56DFXSystem" network_interface="$(arg network_interface)" command_topic="$(arg inspire_command_topic)" state_topic="$(arg inspire_state_topic)" state_timeout_sec="$(arg inspire_state_timeout_sec)"/>
+  <xacro:inspire_rh56dfx_ros2_control name="InspireRH56DFXSystem" network_interface="$(arg network_interface)" command_topic="$(arg inspire_command_topic)" state_topic="$(arg inspire_state_topic)" state_timeout_sec="$(arg inspire_state_timeout_sec)" close_hand_on_deactivate="$(arg close_hand_on_deactivate)"/>
 </robot>

File: g1_hardware/config/inspire_rh56dfx_real.ros2_control.xacro (robot description, xacro)
@@ -8,5 +8,5 @@
       RH56DFX DDS q values are normalized as 0.0 = closed, 1.0 = open.
     -->
-  <xacro:macro name="inspire_rh56dfx_ros2_control" params="name network_interface:='' command_topic:='rt/inspire/cmd' state_topic:='rt/inspire/state' state_timeout_sec:=3.0">
+  <xacro:macro name="inspire_rh56dfx_ros2_control" params="name network_interface:='' command_topic:='rt/inspire/cmd' state_topic:='rt/inspire/state' state_timeout_sec:=3.0 close_hand_on_deactivate:=true">
     <ros2_control name="${name}" type="system">
       <hardware>
@@ -16,4 +16,5 @@
         <param name="state_topic">${state_topic}</param>
         <param name="state_timeout_sec">${state_timeout_sec}</param>
+        <param name="close_hand_on_deactivate">${close_hand_on_deactivate}</param>
       </hardware>
       <!-- Right RH56DFX hand - actuated joints only (URDF mimic joints excluded) -->
